File: src/Custom-ESP32-S3.kicad_pcb (KiCad board)
At the start: 4 copper layers, 79 x 68.9 mm, 77 parts, among them J1 Conn_01x04_Pin, J2 USB_C_Receptacle_USB2.0_16P, J3 Conn_01x18_Pin, J5 Conn_01x04_Pin, J6 Conn_01x02_Pin, J7 Conn_01x18_Pin, Q2 AO3401A, U1 HS96L03W2C03, U2 AMS1117-3.3, U3 W25Q128JVS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

Commit message: Add files via upload
Parts:
- moved AE1 3.72 mm to (152.8, 86.0)
Routing:
- net GND: track 107.4 -> 109.4 mm, vias 33 -> 44
- net Net-(AE1-FEED): track 7.47 -> 8.17 mm
- added copper zone on In1.Cu, net GND
- removed copper zone on In2.Cu, net GND
Other:
- board size 79 x 68.9 mm -> 79.2 x 72.4 mm

Commit message: Add files via upload
Other:
- board size 79.2 x 72.4 mm -> 80 x 73 mm
Changed lines of the file:
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@@
 		(capping no)
 		(filling no)
-		(zone_defaults)
 		(pcbplotparams
 			(layerselection 0x00000000_00000000_55555555_5755f5ff)
@@
 		(embedded_fonts no)
 	)
-	(gr_line
-		(start 119.75 142.075091)
-		(end 120.006757 79.6)
+	(gr_arc
+		(start 120 79)
+		(mid 121.464466 75.464466)
+		(end 125 74)
 		(stroke
 			(width 0.05)
@@
 		(layer "Edge.Cuts")
 	)
-	(gr_arc
-		(start 119.937922 79.733144)
-		(mid 121.4 76.2)
-		(end 124.931165 74.733148)
+	(gr_line
+		(start 120 142)
+		(end 120 79)
 		(stroke
 			(width 0.05)
@@
 		(layer "Edge.Cuts")
 	)
-	(gr_arc
-		(start 124.771969 147.075043)
-		(mid 121.222245 145.618383)
-		(end 119.75 142.075091)
+	(gr_line
+		(start 125 74)
+		(end 195 74)
 		(stroke
 			(width 0.05)
@@
 		(layer "Edge.Cuts")
 	)
-	(gr_line
-		(start 124.95 74.725)
-		(end 193.956757 74.631748)
+	(gr_arc
+		(start 125 147)
+		(mid 121.464466 145.535534)
+		(end 120 142)
 		(stroke
 			(width 0.05)
@@
 		(layer "Edge.Cuts")
 	)
-	(gr_line
-		(start 193.771969 146.771872)
-		(end 124.771969 147.075043)
+	(gr_arc
+		(start 195 74)
+		(mid 198.535534 75.464466)
+		(end 200 79)
 		(stroke
 			(width 0.05)
@@
 		(layer "Edge.Cuts")
 	)
-	(gr_arc
-		(start 193.956757 74.631748)
-		(mid 197.517008 76.095093)
-		(end 198.993285 79.65)
+	(gr_line
+		(start 195 147)
+		(end 125 147)
 		(stroke
 			(width 0.05)
@@
 		(layer "Edge.Cuts")
 	)
-	(gr_arc
-		(start 198.75 141.771921)
-		(mid 197.293285 145.299666)
-		(end 193.771969 146.771872)
+	(gr_line
+		(start 200 79)
+		(end 200 142)
 		(stroke
 			(width 0.05)
@@
 		(layer "Edge.Cuts")
 	)
-	(gr_line
-		(start 198.993285 79.65)
-		(end 198.75 141.771921)
+	(gr_arc
+		(start 200 142)
+		(mid 198.535534 145.535534)
+		(end 195 147)
 		(stroke
 			(width 0.05)
@@
 		(polygon
 			(pts
-				(xy 105 55) (xy 220 57.5) (xy 220 160) (xy 100 165)
+				(xy 105 60) (xy 220.104967 59.90332) (xy 220.18886 159.783618) (xy 103 160)
 			)
 		)
