File: src/kicad/Custom-ESP32-S3.kicad_sch (KiCad schematic)
At the start: 77 parts, among them J1 Conn_01x04_Pin, J2 USB_C_Receptacle_USB2.0_16P, J3 Conn_01x18_Pin, J5 Conn_01x04_Pin, J6 Conn_01x02_Pin, J7 Conn_01x18_Pin, Q2 AO3401A, U1 HS96L03W2C03, U2 AMS1117-3.3, U3 W25Q128JVS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

Commit message: Add files via upload
Other:
- moved on the sheet: C7, C8
